File: pcb tings/pcb tings.kicad_sch (KiCad schematic)
At the start: 24 parts, among them SW1 SW_Push, U1 ATmega32U4-A, Y1 16MHz

Commit message: started working on pcb layout
Connections:
- net COL0: now also MX3.1 (COL); no longer MX2.1 (COL)
- net COL1: now also MX2.1 (COL); no longer MX3.1 (COL)
- net at D3.1 (K): now also D4.1 (K); no longer D1.1 (K)
- net at D2.1 (K): now also D1.1 (K); no longer D4.1 (K)
Other:
- moved on the sheet: D2, D3, MX2, MX3
